File: Barboni!/schema elettrico.kicad_sch (KiCad schematic)
At the start: 27 parts, among them J1 Raspberry_Pi_4, J2 DIN-5, J3 DIN-5, P1 Power Supply, Q1 PNP, SW1 Encoder 1, SW2 Encoder 2, SW3 Encoder 3, SW4 SW_Push, SW5 SW_Push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

Commit message: ttt
Parts:
- added C1, C2: 47microfarad, symbol Device:C_Polarized
- added D3, D5: 1N4148, Diode_THT:D_DO-35_SOD27_P7.62mm_Horizontal, symbol Diode:1N4148
Connections:
- net GND: now also C1.2, C2.2
- net at R13.2: now also D5.2 (A); no longer D4.2 (A)
- net at R8.1: now also C1.1, D3.1 (K); no longer Q1.1 (C)
- new net: C2.1, D4.2 (A), D5.1 (K)
- new net: D3.2 (A), Q1.1 (C)
Other:
- moved on the sheet: D1, D4, R13, R8

Commit message: update, non ci siamo ancora
Parts:
- added Q2: PNP, symbol Simulation_SPICE:PNP
- added R1: 470, Resistor_THT:R_Axial_DIN0204_L3.6mm_D1.6mm_P7.62mm_Horizontal, symbol Device:R_US
Connections:
- net +3.3V: now also Q2.3 (E)
- net GND: no longer U3.6 (GND)
- net at U3.5 (MISO): no longer J1.21 (MISO_SPI0/GPIO09)
- net at J1.35 (GPIO19/SPI1_MISO/PCM_FS): now also R1.1; no longer U3.8 (LED_BL)
- new net: Q2.2 (B), R1.2
- new net: Q2.1 (C), U3.8 (LED_BL)
- new net GND (pin 9): U3.6 (GND)

Commit message: spigolature
Connections:
- net GND (pin 9): now also U3.2 (GND); no longer U3.6 (GND)
- net at J1.24 (~{CE0}_SPI0/GPIO08): now also U3.3 (CS); no longer U3.2 (CS)
- net at J1.31 (GPCLK2/GPIO06): now also U3.4 (O_RESET); no longer U3.3 (O_RESET)
- net at J1.19 (MOSI_SPI0/GPIO10): now also U3.6 (MOSI); no longer U3.4 (MOSI)
- net at U3.5 (O_DC[RS]): now also J1.29 (GPCLK1/GPIO05)
- net at J1.23 (SCLK_SPI0/GPIO11): now also U3.7 (SCK); no longer U3.6 (GND)
Changed lines of the file:
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@@
 		(pin "3"
 		)
-		(pin "6"
+		(pin "9"
 		)
 		(pin "8"
