File: Barboni!/Schema elettrificato/Norns/Norns.kicad_pcb (KiCad board)
At the start: 4 copper layers, 0 parts

Commit message: gerb
Parts:
- added C1: 4,7mF, Capacitor_THT:C_Radial_D5.0mm_H11.0mm_P2.00mm, F.Cu at (153.6, 110.8)
- added C2: 100nF, Capacitor_THT:C_Disc_D5.0mm_W2.5mm_P5.00mm, F.Cu at (152.6, 106.5)
- added C3: 100nF, Capacitor_THT:C_Disc_D5.0mm_W2.5mm_P5.00mm, F.Cu at (127.3, 106.0)
- added C4: 4,7mF, Capacitor_THT:C_Radial_D5.0mm_H11.0mm_P2.00mm, F.Cu at (128.8, 111.2)
- added D1: 1N4148, Diode_THT:D_DO-35_SOD27_P7.62mm_Horizontal, F.Cu at (164.6, 112.5)
- added D2: LED Out, LED_THT:LED_D5.0mm, F.Cu at (171.6, 103.2)
- added D3: 1N4148, Diode_THT:D_DO-35_SOD27_P7.62mm_Horizontal, F.Cu at (173.4, 77.2)
- added D4: 1N4148, Diode_THT:D_DO-35_SOD27_P7.62mm_Horizontal, F.Cu at (139.6, 112.2)
- added D5: LED In, LED_THT:LED_D5.0mm, F.Cu at (145.3, 102.8)
- added D7: LED Pwr, LED_THT:LED_D5.0mm, F.Cu at (125.0, 86.0)
- added J1: MIDI_Din, Connector_PinHeader_2.54mm:PinHeader_1x02_P2.54mm_Vertical, F.Cu at (178.2, 72.2)
- added J2: MIDI_Din, Connector_PinHeader_2.54mm:PinHeader_1x02_P2.54mm_Vertical, F.Cu at (178.0, 87.5)
- added J4: Power Supply, Connector_JST:JST_EH_B2B-EH-A_1x02_P2.50mm_Vertical, F.Cu at (121.2, 70.2)
- added J6: Display, Connector_JST:JST_EH_B8B-EH-A_1x08_P2.50mm_Vertical, F.Cu at (133.0, 78.0)
- added J7: RPi_GPIO, RPI_Hat:RPI_Hat_B+_NoCamera, F.Cu at (149.7, 63.7)
- added J8: Encoders, Connector_JST:JST_EH_B12B-EH-A_1x12_P2.50mm_Vertical, F.Cu at (132.5, 71.0)
- added Q1: 2N2222, Package_TO_SOT_THT:TO-92_Inline, F.Cu at (135.5, 96.5)
- added Q3: 2N2222, Package_TO_SOT_THT:TO-92_Inline, F.Cu at (161.0, 97.5)
- added Q4: S8550, Package_TO_SOT_THT:TO-92_Inline, F.Cu at (153.0, 84.0)
- added R1: 1000, Resistor_THT:R_Axial_DIN0204_L3.6mm_D1.6mm_P5.08mm_Horizontal, F.Cu at (168.9, 108.0)
- added R10: 10000, Resistor_THT:R_Axial_DIN0204_L3.6mm_D1.6mm_P5.08mm_Horizontal, F.Cu at (142.9, 111.0)
- added R11: 220, Resistor_THT:R_Axial_DIN0204_L3.6mm_D1.6mm_P5.08mm_Horizontal, F.Cu at (174.4, 69.4)
- added R12: 220, Resistor_THT:R_Axial_DIN0204_L3.6mm_D1.6mm_P5.08mm_Horizontal, F.Cu at (168.9, 72.9)
- added R13: 1000, Resistor_THT:R_Axial_DIN0204_L3.6mm_D1.6mm_P5.08mm_Horizontal, F.Cu at (142.2, 96.2)
- added R14: 470, Resistor_THT:R_Axial_DIN0204_L3.6mm_D1.6mm_P5.08mm_Horizontal, F.Cu at (157.0, 77.0)
- added R15: 10000, Resistor_THT:R_Axial_DIN0204_L3.6mm_D1.6mm_P5.08mm_Horizontal, F.Cu at (166.2, 88.7)
- added R2: 10000, Resistor_THT:R_Axial_DIN0204_L3.6mm_D1.6mm_P5.08mm_Horizontal, F.Cu at (168.9, 112.0)
- added R3: 1000, Resistor_THT:R_Axial_DIN0204_L3.6mm_D1.6mm_P5.08mm_Horizontal, F.Cu at (152.0, 97.5)
- added R4: 1000, Resistor_THT:R_Axial_DIN0204_L3.6mm_D1.6mm_P5.08mm_Horizontal, F.Cu at (168.5, 96.8)
- added R5: 220, Resistor_THT:R_Axial_DIN0204_L3.6mm_D1.6mm_P5.08mm_Horizontal, F.Cu at (178.0, 77.0)
- added R6: 470, Resistor_THT:R_Axial_DIN0204_L3.6mm_D1.6mm_P5.08mm_Horizontal, F.Cu at (174.2, 88.7)
- added R7: 1000, Resistor_THT:R_Axial_DIN0204_L3.6mm_D1.6mm_P5.08mm_Horizontal, F.Cu at (124.0, 94.0)
- added R8: 1000, Resistor_THT:R_Axial_DIN0204_L3.6mm_D1.6mm_P5.08mm_Horizontal, F.Cu at (126.7, 97.0)
- added R9: 1000, Resistor_THT:R_Axial_DIN0204_L3.6mm_D1.6mm_P5.08mm_Horizontal, F.Cu at (143.0, 108.0)
- added U1: NE555P, Package_DIP:DIP-8_W7.62mm, F.Cu at (164.8, 100.8)
- added U2: 7404, Package_DIP:DIP-14_W7.62mm, F.Cu at (146.5, 83.4)
- added U3: 6N138, Package_DIP:DIP-8_W7.62mm_LongPads, F.Cu at (168.8, 77.2)
- added U4: NE555P, Package_DIP:DIP-8_W7.62mm, F.Cu at (139.8, 100.0)
Routing:
- net +5V: track 0.00 -> 155.2 mm
- net +3.3V: track 0.00 -> 71.5 mm
- net Net-(J7-BCM15_RXD): track 0.00 -> 66.9 mm
- net Net-(J7-BCM21_SCLK_PCM_DO): track 0.00 -> 47.5 mm
- net Net-(R12-Pad1): track 0.00 -> 39.1 mm
- net /CLK3: track 0.00 -> 34.8 mm
- net /O_RESET: track 0.00 -> 34.6 mm
- net /CS: track 0.00 -> 31.5 mm
- net /SW3: track 0.00 -> 31.3 mm
- net Net-(J7-BCM14_TXD): track 0.00 -> 27.3 mm
- net /CLK1: track 0.00 -> 23.2 mm
- net /O_DC: track 0.00 -> 21.7 mm
- net Net-(D1-A): track 0.00 -> 21.0 mm
- net /SW2: track 0.00 -> 20.8 mm
- net Net-(D1-K): track 0.00 -> 20.1 mm
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- added copper zone on B.Cu, net GND
- added copper zone on F.Cu, net GND
Other:
- board outline added: 65 x 56.5 mm
