File: Barboni!/Schema elettrificato/Norns/Norns.kicad_pcb (KiCad board)
At the start: 4 copper layers, 65 x 56.5 mm, 38 parts, among them J1 MIDI_Din, J2 MIDI_Din, J4 Power Supply, J6 Display, J7 RPi_GPIO, J8 Encoders, Q1 2N2222, Q3 2N2222, Q4 S8550, U1 NE555P, U2 7404, U3 6N138, U4 NE555P

Commit message: avanzamento di progressione
Parts:
- MIDI In: renamed from J2
- MIDI Out: renamed from J1
- renumbered D7 to Power
Other:
- board text added: "+ Power -"
- board text added: "JLC p/n"
- board text added: "JLCJLCJLCJLC"
- board text added: "XOR Rev 1.0"
Changed lines of the file:
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@@
 		(pcbplotparams
 			(layerselection 0x00000000_00000000_55555555_5755f5ff)
-			(plot_on_all_layers_selection 0x00000000_00000000_00000000_00000000)
+			(plot_on_all_layers_selection 0x00000000_00000000_00000000_00000020)
 			(disableapertmacros no)
 			(usegerberextensions no)
@@
 			(outputformat 1)
 			(mirror no)
-			(drillshape 1)
+			(drillshape 0)
 			(scaleselection 1)
 			(outputdirectory "")
@@
 			(layer "F.Fab")
 		)
-		(fp_text user "${REFERENCE}"
-			(at 1.27 0 90)
-			(layer "F.Fab")
+		(fp_text user "Led Out"
+			(at 1.27 3.44 90)
+			(layer "F.SilkS")
 			(effects
 				(font
@@
 			(layer "F.Fab")
 		)
-		(fp_text user "${REFERENCE}"
-			(at 8.75 1.5 0)
-			(layer "F.Fab")
+		(fp_text user "Display"
+			(at 8.75 3 0)
+			(layer "F.SilkS")
 			(effects
 				(font
@@
 		(descr "Through hole straight pin header, 1x02, 2.54mm pitch, single row")
 		(tags "Through hole pin header THT 1x02 2.54mm single row")
-		(property "Reference" "J1"
-			(at 0 -2.38 0)
+		(property "Reference" "MIDI Out"
+			(at -1.81 1.19 90)
 			(layer "F.SilkS")
 			(effects
@@
 		(descr "LED, diameter 5.0mm, 2 pins, http://cdn-reichelt.de/documents/datenblatt/A500/LL-504BC2E-009.pdf, generated by kicad-footprint-generator")
 		(tags "LED")
-		(property "Reference" "D7"
-			(at 1.27 -2.5 90)
+		(property "Reference" "Power"
+			(at -4 0 90)
 			(layer "F.SilkS")
 			(effects
@@
 		(descr "Through hole straight pin header, 1x02, 2.54mm pitch, single row")
 		(tags "Through hole pin header THT 1x02 2.54mm single row")
-		(property "Reference" "J2"
-			(at 0 -2.38 0)
+		(property "Reference" "MIDI In"
+			(at 2 2.54 90)
 			(layer "F.SilkS")
 			(effects
@@
 			(layer "F.Fab")
 		)
-		(fp_text user "${REFERENCE}"
-			(at 13.75 1.5 0)
-			(layer "F.Fab")
+		(fp_text user "Buttons and Encoders"
+			(at 13.5 3 0)
+			(layer "F.SilkS")
 			(effects
 				(font
@@
 			(layer "F.Fab")
 		)
-		(fp_text user "${REFERENCE}"
-			(at 1.27 0 90)
-			(layer "F.Fab")
+		(fp_text user "Led In"
+			(at 1.27 3.69 90)
+			(layer "F.SilkS")
 			(effects
 				(font
@@
 			)
 		)
-		(pad "1" thru_hole roundrect
+		(pad "1" thru_hole oval
 			(at 0 0)
 			(size 1.7 2)
@@
 			(layers "*.Cu" "*.Mask")
 			(remove_unused_layers no)
-			(roundrect_rratio 0.147059)
 			(net 2 "+5V")
 			(pinfunction "Pin_1")
 			(pintype "power_out")
 		)
-		(pad "2" thru_hole oval
+		(pad "2" thru_hole roundrect
 			(at 2.5 0)
 			(size 1.7 2)
@@
 			(layers "*.Cu" "*.Mask")
 			(remove_unused_layers no)
+			(roundrect_rratio 0.1470588235)
 			(net 1 "GND")
 			(pinfunction "Pin_2")
@@
 		)
 	)
+	(gr_circle
+		(center 179.57 73.57)
+		(end 179.14 73.9975)
+		(stroke
+			(width 0.1)
+			(type solid)
+		)
+		(fill yes)
+		(layer "F.SilkS")
+	)
+	(gr_circle
+		(center 179.27 86.19)
+		(end 180 86.19)
+		(stroke
+			(width 0.1)
+			(type solid)
+		)
+		(fill yes)
+		(layer "F.SilkS")
+	)
+	(gr_text "+ Power -"
+		(at 118 74 0)
+		(layer "F.SilkS")
+		(effects
+			(font
+				(size 1 1)
+				(thickness 0.15)
+			)
+			(justify left bottom)
+		)
+	)
+	(gr_text "XOR Rev 1.0"
+		(at 120 109 90)
+		(layer "F.SilkS")
+		(effects
+			(font
+				(size 1 1)
+				(thickness 0.15)
+			)
+			(justify left bottom)
+		)
+	)
+	(gr_text "JLC p/n"
+		(at 124 115 90)
+		(layer "F.SilkS")
+		(effects
+			(font
+				(size 0.8128 0.8128)
+				(thickness 0.1524)
+				(bold yes)
+			)
+			(justify left bottom)
+		)
+	)
+	(gr_text "JLCJLCJLCJLC"
+		(at 124 109 90)
+		(layer "F.SilkS")
+		(effects
+			(font
+				(size 0.8128 0.8128)
+				(thickness 0.1524)
+				(bold yes)
+			)
+			(justify left bottom)
+		)
+	)

Commit message: schema el
Parts:
- removed C3: 100nF, Capacitor_THT:C_Disc_D5.0mm_W2.5mm_P5.00mm
- removed C4: 4,7mF, Capacitor_THT:C_Radial_D5.0mm_H11.0mm_P2.00mm
- removed J7: RPi_GPIO, RPI_Hat:RPI_Hat_B+_NoCamera
- removed J8: Encoders, Connector_JST:JST_EH_B12B-EH-A_1x12_P2.50mm_Vertical
- removed MIDI In: MIDI_Din, Connector_PinHeader_2.54mm:PinHeader_1x02_P2.54mm_Vertical
- removed MIDI Out: MIDI_Din, Connector_PinHeader_2.54mm:PinHeader_1x02_P2.54mm_Vertical
- removed Power: LED Pwr, LED_THT:LED_D5.0mm
- removed Q4: S8550, Package_TO_SOT_THT:TO-92_Inline
- removed R12: 220, Resistor_THT:R_Axial_DIN0204_L3.6mm_D1.6mm_P5.08mm_Horizontal
- removed R13: 1000, Resistor_THT:R_Axial_DIN0204_L3.6mm_D1.6mm_P5.08mm_Horizontal
- removed R14: 470, Resistor_THT:R_Axial_DIN0204_L3.6mm_D1.6mm_P5.08mm_Horizontal
- removed R15: 10000, Resistor_THT:R_Axial_DIN0204_L3.6mm_D1.6mm_P5.08mm_Horizontal
- removed U3: 6N138, Package_DIP:DIP-8_W7.62mm_LongPads
- removed U4: NE555P, Package_DIP:DIP-8_W7.62mm
- added D6: LED Out, LED_THT:LED_D5.0mm, F.Cu at (153.0, 92.8)
- added J1: Power Supply, Connector_JST:JST_EH_B2B-EH-A_1x02_P2.50mm_Vertical, F.Cu at (91.5, 51.0)
- added J2: RPi_GPIO, RPI_Hat:RPI_Hat_B+_NoCamera, F.Cu at (117.4, 44.1)
- added J3: Display, Connector_JST:JST_EH_B8B-EH-A_1x08_P2.50mm_Vertical, F.Cu at (106.5, 56.0)
- added J5: MIDI_Din, Connector_PinHeader_2.54mm:PinHeader_1x02_P2.54mm_Vertical, F.Cu at (138.5, 111.1)
- added Q2: 2N7000, Package_TO_SOT_THT:TO-92_Inline, F.Cu at (131.7, 106.2)
- C1: value 4,7mF -> 2,2 mF
- C2: value 100nF -> 2,2 mF; footprint Capacitor_THT:C_Disc_D5.0mm_W2.5mm_P5.00mm -> Capacitor_THT:C_Radial_D5.0mm_H11.0mm_P2.00mm
- D1: value 1N4148 -> LED Pwr; footprint Diode_THT:D_DO-35_SOD27_P7.62mm_Horizontal -> LED_THT:LED_D5.0mm
- D2: value LED Out -> 1N4148; footprint LED_THT:LED_D5.0mm -> Diode_THT:D_DO-35_SOD27_P7.62mm_Horizontal
- D5: value LED In -> LED Out
- J4: value Power Supply -> Encoders; footprint Connector_JST:JST_EH_B2B-EH-A_1x02_P2.50mm_Vertical -> Connector_JST:JST_EH_B12B-EH-A_1x12_P2.50mm_Vertical
- J6: value Display -> MIDI_Din; footprint Connector_JST:JST_EH_B8B-EH-A_1x08_P2.50mm_Vertical -> Connector_PinHeader_2.54mm:PinHeader_1x02_P2.54mm_Vertical
- Q1: value 2N2222 -> S8550
- Q3: value 2N2222 -> 2N7000
- R1, R3: value 1000 -> 470
- R10, R2: value 10000 -> 1000
- R11: value 220 -> 1000
- R4: value 1000 -> 10000
- R6: value 470 -> 220
- R7: value 1000 -> 220
- R8, R9: value 1000 -> 100K
- U1: value NE555P -> 7404; footprint Package_DIP:DIP-8_W7.62mm -> Package_DIP:DIP-14_W7.62mm
- U2: value 7404 -> 6N138; footprint Package_DIP:DIP-14_W7.62mm -> Package_DIP:DIP-8_W7.62mm_LongPads
- moved R2 69.8 mm to (152.0, 44.2)
- moved R1 62.2 mm to (138.0, 54.0), turned to -90 degrees
- moved U1 58.3 mm to (112.5, 75.0)
- moved R3 50.1 mm to (152.0, 47.4)
- moved R4 49.1 mm to (152.0, 50.5)
- moved R7 44.0 mm to (152.0, 60.0), turned to 0 degrees
- moved R9 42.7 mm to (152.0, 66.3)
- moved C1 42.6 mm to (111.2, 106.2), turned to 0 degrees
- moved R10 42.5 mm to (152.0, 69.5)
- moved R8 42.2 mm to (152.0, 63.1)
- moved C2 41.8 mm to (111.2, 112.8), turned to 0 degrees
- moved Q1 41.6 mm to (132.0, 55.0), turned to -90 degrees
- moved R6 38.8 mm to (152.0, 56.9), turned to 0 degrees
- moved D1 36.5 mm to (153.0, 77.9), turned to 0 degrees
- moved R5 34.9 mm to (152.0, 53.7), turned to 0 degrees
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Connections:
- C1 pad 1: Net-(D1-A) -> Net-(D3-K)
- C2 pad 1: Net-(U1-CV) -> Net-(D4-K)
- D1 pad 1: Net-(D1-K) -> GND
- D2 pad 1: GND -> Net-(D2-K)
- J4 pad 1: +5V -> +3.3V
- J4 pad 2: GND -> unconnected-(J4-Pin_2-Pad2)
- J6 pad 1: +3.3V -> Net-(J6-Pad1)
- J6 pad 2: /CS -> Net-(J6-Pad2)
- Q1 pad 1: GND -> /LED_BL
- Q1 pad 3: Net-(D4-K) -> +3.3V
- Q3 pad 2: Net-(Q3-B) -> Net-(D4-K)
- Q3 pad 3: Net-(D1-K) -> Net-(Q3-D)
- R1 pad 1: Net-(D1-K) -> Net-(J2-BCM19_MISO_PCM_FS)
- R1 pad 2: +5V -> Net-(Q1-B)
- R10 pad 1: Net-(D4-A) -> Net-(Q2-D)
- R10 pad 2: +5V -> Net-(D5-A)
- R11 pad 1: Net-(J1-Pad2) -> Net-(Q3-D)
- R11 pad 2: +5V -> Net-(D6-A)
- R2 pad 2: +5V -> Net-(R2-Pad2)
- R3 pad 1: Net-(R3-Pad1) -> +3.3V
- R3 pad 2: Net-(Q3-B) -> Net-(J2-BCM15_RXD)
- R4 pad 1: Net-(U1-Q) -> Net-(U2-VO1)
- R4 pad 2: Net-(D2-A) -> GND
- R5 pad 1: Net-(D3-K) -> Net-(D2-K)
- R6 pad 1: +3.3V -> Net-(R6-Pad1)
- R6 pad 2: Net-(J7-BCM15_RXD) -> Net-(J6-Pad1)
- R7 pad 1: Net-(D7-A) -> Net-(J6-Pad2)
- R7 pad 2: Net-(R7-Pad2) -> +5V
- R8 pad 1: Net-(R8-Pad1) -> GND
- R8 pad 2: Net-(Q1-B) -> Net-(D3-K)
- R9 pad 1: Net-(D4-K) -> GND
- R9 pad 2: +5V -> Net-(D4-K)
- U1 pad 1: GND -> Net-(J2-BCM14_TXD)
- U1 pad 2: Net-(D1-K) -> Net-(D3-A)
- U1 pad 3: Net-(U1-Q) -> Net-(D3-A)
- U1 pad 4: +5V -> Net-(R6-Pad1)
- U1 pad 5: Net-(U1-CV) -> Net-(J2-BCM21_SCLK_PCM_DO)
- U1 pad 6: Net-(D1-A) -> Net-(R2-Pad2)
- U1 pad 7: Net-(D1-A) -> GND
- U1 pad 8: +5V -> Net-(D4-A)
- U2 pad 1: Net-(J7-BCM14_TXD) -> unconnected-(U2-NC-Pad1)
- U2 pad 2: Net-(R3-Pad1) -> Net-(D2-K)
- U2 pad 3: Net-(R3-Pad1) -> Net-(D2-A)
- U2 pad 4: Net-(R12-Pad1) -> unconnected-(U2-NC-Pad4)
- U2 pad 5: Net-(J7-BCM21_SCLK_PCM_DO) -> GND
- U2 pad 6: Net-(R7-Pad2) -> Net-(J2-BCM15_RXD)
- U2 pad 7: GND -> Net-(U2-VO1)
- U2 pad 8: Net-(R8-Pad1) -> +3.3V
Routing:
- net +5V: track 155.2 -> 8.85 mm
- net Net-(J7-BCM15_RXD): track 66.9 -> 0.00 mm
- net Net-(J7-BCM21_SCLK_PCM_DO): track 47.5 -> 0.00 mm
- net Net-(R12-Pad1): track 39.1 -> 0.00 mm
- net Net-(J7-BCM14_TXD): track 27.3 -> 0.00 mm
- net /Data3: track 15.1 -> 36.7 mm
- net /CLK2: track 9.03 -> 30.2 mm
- net Net-(D1-A): track 21.0 -> 0.00 mm
- net Net-(D1-K): track 20.1 -> 0.00 mm
- net Net-(R3-Pad1): track 20.0 -> 0.00 mm
- net Net-(D3-A): track 19.9 -> 0.00 mm
- net Net-(D4-K): track 19.9 -> 0.00 mm
- net Net-(R7-Pad2): track 19.8 -> 0.00 mm
- net Net-(D4-A): track 18.9 -> 0.00 mm
- net Net-(J7-BCM19_MISO_PCM_FS): track 16.8 -> 0.00 mm
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- removed copper zone on B.Cu, net GND
- removed copper zone on F.Cu, net GND
Other:
- board text removed: "+ Power -"
- board text removed: "JLC p/n"
- board text removed: "JLCJLCJLCJLC"
- board text removed: "XOR Rev 1.0"

Commit message: a
Parts:
- added J7: MIDI_Din, Connector_PinHeader_2.54mm:PinHeader_1x02_P2.54mm_Vertical, F.Cu at (185.4, 120.5)
- added J8: MIDI_Din, Connector_PinHeader_2.54mm:PinHeader_1x02_P2.54mm_Vertical, F.Cu at (190.0, 120.5)
- J1: value Power Supply -> Display; footprint Connector_JST:JST_EH_B2B-EH-A_1x02_P2.50mm_Vertical -> Connector_JST:JST_EH_B8B-EH-A_1x08_P2.50mm_Vertical
- J2: value RPi_GPIO -> Encoder 1; footprint RPI_Hat:RPI_Hat_B+_NoCamera -> Connector_JST:JST_EH_B5B-EH-A_1x05_P2.50mm_Vertical
- J3: value Display -> Power Supply; footprint Connector_JST:JST_EH_B8B-EH-A_1x08_P2.50mm_Vertical -> Connector_JST:JST_EH_B2B-EH-A_1x02_P2.50mm_Vertical
- J4: value Encoders -> RPi_GPIO; footprint Connector_JST:JST_EH_B12B-EH-A_1x12_P2.50mm_Vertical -> RPI_Hat:RPI_Hat_B+_NoCamera
- J5: value MIDI_Din -> Encoder 2; footprint Connector_PinHeader_2.54mm:PinHeader_1x02_P2.54mm_Vertical -> Connector_JST:JST_EH_B5B-EH-A_1x05_P2.50mm_Vertical
- J6: value MIDI_Din -> Encoder 3; footprint Connector_PinHeader_2.54mm:PinHeader_1x02_P2.54mm_Vertical -> Connector_JST:JST_EH_B5B-EH-A_1x05_P2.50mm_Vertical
- moved Q1 72.6 mm to (172.0, 115.6), turned to 0 degrees
- moved C1 69.5 mm to (178.8, 122.1)
- moved C2 67.7 mm to (178.8, 115.6)
- moved J1 65.7 mm to (150.5, 80.0)
- moved U1 50.3 mm to (143.8, 114.4), turned to 0 degrees
- moved J4 49.2 mm to (150.7, 59.3)
- moved R1 47.3 mm to (185.2, 56.3), turned to 0 degrees
- moved Q2 45.5 mm to (172.0, 127.2)
- moved J6 44.8 mm to (163.0, 71.0)
- moved Q3 41.4 mm to (172.0, 121.4)
- moved J5 40.6 mm to (145.0, 71.0)
- moved D5 40.3 mm to (186.2, 108.0)
- moved R10 38.0 mm to (185.2, 87.8)
- moved R8 38.0 mm to (185.2, 81.5)
- moved R3 36.6 mm to (185.2, 62.6)
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Connections:
- D5 pad 1: GND -> Net-(D5-K)
- D6 pad 1: GND -> Net-(D6-K)
- J1 pad 1: +5V -> +3.3V
- J1 pad 2: GND -> /CS
- J2 pad 2: +5V -> /Data
- J2 pad 3: unconnected-(J2-BCM2_SDA-Pad3) -> /Clock
- J2 pad 4: unconnected-(J2-5V-Pad4) -> /Switch
- J2 pad 5: unconnected-(J2-BCM3_SCL-Pad5) -> GND
- J3 pad 1: +3.3V -> +5V
- J3 pad 2: /CS -> GND
- J4 pad 10: /Data1 -> Net-(J4-BCM15_RXD)
- J4 pad 11: /SW1 -> unconnected-(J4-BCM17-Pad11)
- J4 pad 12: GND -> unconnected-(J4-BCM18_PCM_C-Pad12)
- J4 pad 2: unconnected-(J4-Pin_2-Pad2) -> +5V
- J4 pad 3: /CLK3 -> unconnected-(J4-BCM2_SDA-Pad3)
- J4 pad 4: /Data3 -> unconnected-(J4-5V-Pad4)
- J4 pad 5: /SW3 -> unconnected-(J4-BCM3_SCL-Pad5)
- J4 pad 6: /CLK2 -> GND
- J4 pad 7: /Data2 -> /Clock
- J4 pad 8: /SW2 -> Net-(J4-BCM14_TXD)
- J4 pad 9: /CLK1 -> GND
- J5 pad 1: Net-(J5-Pad1) -> +3.3V
- J5 pad 2: Net-(D2-A) -> /Data2
- J6 pad 1: Net-(J6-Pad1) -> +3.3V
- J6 pad 2: Net-(J6-Pad2) -> /Data3
- Q2 pad 3: Net-(Q2-D) -> Net-(D5-K)
- Q3 pad 3: Net-(Q3-D) -> Net-(D6-K)
- R1 pad 1: Net-(J2-BCM19_MISO_PCM_FS) -> Net-(J4-BCM19_MISO_PCM_FS)
- R10 pad 1: Net-(Q2-D) -> Net-(D5-A)
- R10 pad 2: Net-(D5-A) -> +5V
- R11 pad 1: Net-(Q3-D) -> Net-(D6-A)
- R11 pad 2: Net-(D6-A) -> +5V
- R3 pad 2: Net-(J2-BCM15_RXD) -> Net-(J4-BCM15_RXD)
- R5 pad 2: Net-(J5-Pad1) -> Net-(J7-Pad1)
- R6 pad 2: Net-(J6-Pad1) -> Net-(J8-Pad1)
- R7 pad 1: Net-(J6-Pad2) -> Net-(J8-Pad2)
- U1 pad 1: Net-(J2-BCM14_TXD) -> Net-(J4-BCM14_TXD)
- U1 pad 2: Net-(D3-A) -> Net-(D4-A)
- U1 pad 3: Net-(D3-A) -> Net-(D4-A)
- U1 pad 5: Net-(J2-BCM21_SCLK_PCM_DO) -> Net-(J4-BCM21_SCLK_PCM_DO)
- U1 pad 8: Net-(D4-A) -> Net-(D3-A)
- U1 pad 9: Net-(J2-BCM15_RXD) -> Net-(J4-BCM15_RXD)
- U2 pad 6: Net-(J2-BCM15_RXD) -> Net-(J4-BCM15_RXD)
Routing:
- net +3.3V: track 57.6 -> 0.00 mm
- net /CLK3: track 47.6 -> 0.00 mm
- net /SW3: track 44.7 -> 0.00 mm
- net /SW2: track 33.0 -> 0.00 mm
- net /CLK1: track 30.7 -> 0.00 mm
- net /CLK2: track 30.2 -> 0.00 mm
- net /Data1: track 27.1 -> 0.00 mm
- net /SW1: track 27.1 -> 0.00 mm
- net /Switch2: track 0.00 -> 20.3 mm
- net /Data: track 0.00 -> 19.1 mm
- net /Data3: track 36.7 -> 19.9 mm
- net /Switch: track 0.00 -> 14.5 mm
- net /Clk3: track 0.00 -> 14.3 mm
- net /Clk2: track 0.00 -> 14.2 mm
- net /Data2: track 27.5 -> 14.2 mm
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
Commit message: modifiche
Parts:
- removed D4: 1N4148, Diode_THT:D_DO-35_SOD27_P7.62mm_Horizontal
- removed D5, D6: LED Out, LED_THT:LED_D5.0mm
- removed J7, J8: MIDI_Din, Connector_PinHeader_2.54mm:PinHeader_1x02_P2.54mm_Vertical
- D1: value LED Pwr -> 1N4148; footprint LED_THT:LED_D5.0mm -> Diode_THT:D_DO-35_SOD27_P7.62mm_Horizontal
- J2: value Encoder 1 -> Raspoberro; footprint Connector_JST:JST_EH_B5B-EH-A_1x05_P2.50mm_Vertical -> RPI_Hat:RPI_Hat_B+_No_Camera
- J4: value RPi_GPIO -> Encoders; footprint RPI_Hat:RPI_Hat_B+_NoCamera -> Connector_JST:JST_EH_B12B-EH-A_1x12_P2.50mm_Vertical
- J5: value Encoder 2 -> MIDI; footprint Connector_JST:JST_EH_B5B-EH-A_1x05_P2.50mm_Vertical -> Connector_JST:JST_EH_B4B-EH-A_1x04_P2.50mm_Vertical
- J6: value Encoder 3 -> LED; footprint Connector_JST:JST_EH_B5B-EH-A_1x05_P2.50mm_Vertical -> Connector_JST:JST_EH_B6B-EH-A_1x06_P2.50mm_Vertical
- moved C1 102.8 mm to (94.0, 64.0), turned to -90 degrees
- moved C2 94.7 mm to (94.5, 72.5), turned to -90 degrees
- moved Q2 87.8 mm to (111.5, 63.5), turned to -90 degrees
- moved R8 85.0 mm to (101.5, 67.0)
- moved R9 83.9 mm to (101.5, 74.5)
- moved Q1 79.5 mm to (120.0, 55.5), turned to -90 degrees
- moved Q3 78.8 mm to (111.6, 70.7), turned to -90 degrees
- moved J4 73.4 mm to (86.2, 94.2), turned to 90 degrees
- moved R4 72.4 mm to (119.0, 95.0), turned to 180 degrees
- moved D1 69.6 mm to (118.5, 77.5), turned to 180 degrees
- moved R3 65.8 mm to (128.0, 95.0), turned to 180 degrees
- moved R5 64.8 mm to (121.0, 77.5)
- moved D2 61.3 mm to (106.8, 63.5), turned to 180 degrees
- moved D3 60.9 mm to (107.0, 71.0), turned to 180 degrees
- moved R11 60.9 mm to (127.0, 67.0), turned to -90 degrees
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Connections:
- C1 pad 1: Net-(D3-K) -> Net-(D2-K)
- C2 pad 1: Net-(D4-K) -> Net-(D3-K)
- D1 pad 1: GND -> Net-(D1-K)
- J2 pad 2: /Data -> +5V
- J2 pad 3: /Clock -> unconnected-(J2-BCM2_SDA-Pad3)
- J2 pad 4: /Switch -> unconnected-(J2-5V-Pad4)
- J2 pad 5: GND -> unconnected-(J2-BCM3_SCL-Pad5)
- J4 pad 10: Net-(J4-BCM15_RXD) -> Net-(J2-BCM26)
- J4 pad 12: unconnected-(J4-BCM18_PCM_C-Pad12) -> GND
- J4 pad 2: +5V -> Net-(J2-BCM27)
- J4 pad 3: unconnected-(J4-BCM2_SDA-Pad3) -> Net-(J2-BCM4_GPCLK0)
- J4 pad 4: unconnected-(J4-5V-Pad4) -> Net-(J2-BCM22)
- J4 pad 5: unconnected-(J4-BCM3_SCL-Pad5) -> Net-(J2-BCM23)
- J4 pad 6: GND -> Net-(J2-BCM24)
- J4 pad 7: /Clock -> Net-(J2-BCM13_PWM1)
- J4 pad 8: Net-(J4-BCM14_TXD) -> Net-(J2-BCM25)
- J4 pad 9: GND -> Net-(J2-BCM12_PWM0)
- J5 pad 1: +3.3V -> Net-(J5-Pin_1)
- J5 pad 2: /Data2 -> Net-(J5-Pin_2)
- J5 pad 3: /Clk2 -> Net-(J5-Pin_3)
- J5 pad 4: /Switch2 -> Net-(D1-A)
- J6 pad 1: +3.3V -> Net-(J6-Pin_1)
- J6 pad 2: /Data3 -> Net-(J6-Pin_2)
- J6 pad 3: /Clk3 -> Net-(J6-Pin_3)
- J6 pad 4: /Switch3 -> Net-(J6-Pin_4)
- J6 pad 5: GND -> Net-(J6-Pin_5)
- Q2 pad 2: Net-(D3-K) -> Net-(D2-K)
- Q2 pad 3: Net-(D5-K) -> Net-(J6-Pin_4)
- Q3 pad 2: Net-(D4-K) -> Net-(D3-K)
- Q3 pad 3: Net-(D6-K) -> Net-(J6-Pin_2)
- R1 pad 1: Net-(J4-BCM19_MISO_PCM_FS) -> Net-(J2-BCM19_MISO_PCM_FS)
- R10 pad 1: Net-(D5-A) -> Net-(J6-Pin_3)
- R11 pad 1: Net-(D6-A) -> Net-(J6-Pin_1)
- R2 pad 1: Net-(D1-A) -> Net-(J6-Pin_5)
- R3 pad 2: Net-(J4-BCM15_RXD) -> Net-(J2-BCM15_RXD)
- R5 pad 1: Net-(D2-K) -> Net-(D1-K)
- R5 pad 2: Net-(J7-Pad1) -> Net-(J5-Pin_3)
- R6 pad 2: Net-(J8-Pad1) -> Net-(J5-Pin_1)
- R7 pad 1: Net-(J8-Pad2) -> Net-(J5-Pin_2)
- R8 pad 2: Net-(D3-K) -> Net-(D2-K)
- R9 pad 2: Net-(D4-K) -> Net-(D3-K)
- U1 pad 1: Net-(J4-BCM14_TXD) -> Net-(J2-BCM14_TXD)
- U1 pad 2: Net-(D4-A) -> Net-(D3-A)
- U1 pad 3: Net-(D4-A) -> Net-(D3-A)
- U1 pad 5: Net-(J4-BCM21_SCLK_PCM_DO) -> Net-(J2-BCM21_SCLK_PCM_DO)
- U1 pad 8: Net-(D3-A) -> Net-(D2-A)
- U1 pad 9: Net-(J4-BCM15_RXD) -> Net-(J2-BCM15_RXD)
- U2 pad 2: Net-(D2-K) -> Net-(D1-K)
- U2 pad 3: Net-(D2-A) -> Net-(D1-A)
- U2 pad 6: Net-(J4-BCM15_RXD) -> Net-(J2-BCM15_RXD)
Routing:
- net /O_RESET: track 26.7 -> 0.00 mm
- net /CS: track 24.1 -> 0.00 mm
- net /MOSI: track 22.9 -> 0.00 mm
- net /O_DC: track 22.7 -> 0.00 mm
- net /SCK: track 21.8 -> 0.00 mm
- net /Switch2: track 20.3 -> 0.00 mm
- net /Data3: track 19.9 -> 0.00 mm
- net /Data: track 19.1 -> 0.00 mm
- net /Switch: track 14.5 -> 0.00 mm
- net /Clk3: track 14.3 -> 0.00 mm
- net /Data2: track 14.2 -> 0.00 mm
- net /Clk2: track 14.2 -> 0.00 mm
- net /Clock: track 11.3 -> 0.00 mm
- net /Switch3: track 11.1 -> 0.00 mm
Other:
- copper layers 4 -> 2

Commit message: ola
Parts:
- moved J4 35.6 mm to (75.5, 60.2), turned to -90 degrees
- moved J2 14.8 mm to (97.5, 41.2)
- moved U1 12.8 mm to (97.8, 77.2)
- moved C1 12.4 mm to (83.3, 57.8)
- moved C2 12.4 mm to (83.8, 66.2)
- moved D2 12.4 mm to (96.1, 57.2)
- moved D3 12.4 mm to (96.3, 64.8)
- moved J1 12.4 mm to (84.8, 50.2)
- moved J3 12.4 mm to (72.3, 49.8)
- moved Q1 12.4 mm to (109.3, 49.2)
- moved Q2 12.4 mm to (100.8, 57.2)
- moved Q3 12.4 mm to (100.9, 64.5)
- moved R1 12.4 mm to (115.4, 48.2)
- moved R2 12.4 mm to (120.3, 53.2)
- moved R3 12.4 mm to (117.3, 88.8)
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
Commit message: committamento
Parts:
- C1, C2: footprint Capacitor_THT:C_Radial_D5.0mm_H11.0mm_P2.00mm -> Capacitor_THT:CP_Radial_D5.0mm_P2.50mm
- U2: footprint Package_DIP:DIP-8_W7.62mm_LongPads -> Package_DIP:DIP-8_W7.62mm
- moved R6 38.1 mm to (85.7, 62.8), turned to 0 degrees
- moved R2 33.3 mm to (93.5, 73.0), turned to 90 degrees
- moved D3 26.6 mm to (81.8, 87.0)
- moved D2 26.4 mm to (81.8, 79.5)
- moved R11 26.3 mm to (114.5, 87.0), turned to 180 degrees
- moved Q1 26.3 mm to (83.0, 50.0), turned to 90 degrees
- moved C1 23.8 mm to (88.5, 81.0), turned to 90 degrees
- moved R10 23.0 mm to (114.5, 83.0), turned to 180 degrees
- moved C2 22.4 mm to (88.1, 88.2), turned to 90 degrees
- moved R4 21.8 mm to (109.5, 67.0), turned to 0 degrees
- moved Q3 21.5 mm to (100.0, 86.0)
- moved J5 21.1 mm to (120.5, 61.5)
- moved Q2 20.8 mm to (100.0, 78.0)
- moved J6 18.4 mm to (120.5, 83.5)
- moved R3 18.0 mm to (114.5, 71.0)
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Routing:
- net +5V: track 0.00 -> 106.0 mm
- net +3.3V: track 0.00 -> 81.2 mm
- net Net-(J2-BCM21_SCLK_PCM_DO): track 0.00 -> 68.0 mm
- net Net-(J2-BCM15_RXD): track 0.00 -> 51.2 mm
- net Net-(Q1-B): track 0.00 -> 37.7 mm
- net Net-(J2-BCM14_TXD): track 0.00 -> 37.2 mm
- net Net-(D1-A): track 0.00 -> 30.4 mm
- net Net-(J5-Pin_1): track 0.00 -> 30.3 mm
- net Net-(J6-Pin_5): track 0.00 -> 29.1 mm
- net Net-(D3-A): track 0.00 -> 27.6 mm
- net Net-(J5-Pin_2): track 0.00 -> 26.3 mm
- net Net-(J2-BCM13_PWM1): track 0.00 -> 25.9 mm
- net /LED_BL: track 0.00 -> 25.6 mm
- net Net-(J6-Pin_2): track 0.00 -> 23.6 mm
- net Net-(J6-Pin_4): track 0.00 -> 23.0 mm
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- added copper zone on F.Cu, net GND

Commit message: aricommit
Routing:
- net Net-(J2-BCM15_RXD): track 51.2 -> 75.2 mm
Changed lines of the file:
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@@
 	)
 	(segment
-		(start 106.014949 75.435)
-		(end 109.46 71.989949)
+		(start 82.195 41.453)
+		(end 83.56 40.088)
 		(width 0.25)
-		(layer "F.Cu")
-		(net "Net-(J2-BCM15_RXD)")
-	)
-	(segment
-		(start 109.46 71.989949)
-		(end 109.46 71)
-		(width 0.25)
-		(layer "F.Cu")
-		(net "Net-(J2-BCM15_RXD)")
-	)
-	(segment
-		(start 100.855 75.435)
-		(end 106.014949 75.435)
-		(width 0.25)
-		(layer "F.Cu")
+		(layer "B.Cu")
 		(net "Net-(J2-BCM15_RXD)")
 	)
@@
 		(start 99.73 74.31)
 		(end 100.855 75.435)
-		(width 0.25)
-		(layer "F.Cu")
-		(net "Net-(J2-BCM15_RXD)")
-	)
-	(segment
-		(start 82.195 41.453)
-		(end 83.56 40.088)
 		(width 0.25)
 		(layer "B.Cu")
@@
 	)
 	(segment
+		(start 105.275991 75.435)
+		(end 109.46 71.250991)
+		(width 0.25)
+		(layer "B.Cu")
+		(net "Net-(J2-BCM15_RXD)")
+	)
+	(segment
 		(start 76.92 73.815)
 		(end 76.815 73.815)
@@
 	)
 	(segment
+		(start 97.435 72.015)
+		(end 99.73 74.31)
+		(width 0.25)
+		(layer "B.Cu")
+		(net "Net-(J2-BCM15_RXD)")
+	)
+	(segment
 		(start 79.845 61.679009)
 		(end 79.845 42.141299)
+		(width 0.25)
+		(layer "B.Cu")
+		(net "Net-(J2-BCM15_RXD)")
+	)
+	(segment
+		(start 76.92 73.815)
+		(end 78.72 72.015)
 		(width 0.25)
 		(layer "B.Cu")
@@
 		(width 0.25)
 		(layer "B.Cu")
+		(net "Net-(J2-BCM15_RXD)")
+	)
+	(segment
+		(start 100.855 75.435)
+		(end 105.275991 75.435)
+		(width 0.25)
+		(layer "B.Cu")
+		(net "Net-(J2-BCM15_RXD)")
+	)
+	(segment
+		(start 109.46 71.250991)
+		(end 109.46 71)
+		(width 0.25)
+		(layer "B.Cu")
+		(net "Net-(J2-BCM15_RXD)")
+	)
+	(segment
+		(start 78.72 72.015)
+		(end 97.435 72.015)
+		(width 0.25)
+		(layer "B.Cu")

Commit message: pcb
Other:
- board text added: "${TITLE} Rev. ${REVISION}"
Changed lines of the file:
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@@
 	)
 	(paper "A4")
+	(title_block
+		(title "Trapanaorecchi")
+		(date "2026-06-05")
+		(rev "1.0")
+		(comment 1 "Una libera reinterpretazione del Monome Norns")
+	)
 	(layers
 		(0 "F.Cu" signal)
@@
 		)
 	)
+	(gr_text "${TITLE} Rev. ${REVISION} "
+		(at 108.25 91 0)
+		(layer "F.SilkS")
+		(effects
+			(font
+				(size 1 0.8128)
+				(thickness 0.1524)
+				(bold yes)
+			)
+			(justify left bottom)
+		)
+	)
