File: Barboni!/Schema elettrificato/Norns/collegam_connett.kicad_sch (KiCad schematic)
At the start: 11 parts, among them J1 Conn_01x04, J2 Conn_01x06, J3 MIDI_Din, J4 MIDI_Din, J5 Conn_01x12

Commit message: finito
Connections:
- net at J1.3 (Pin_3): now also J4.2; no longer J4.1
- net at J1.4 (Pin_4): now also J4.1; no longer J4.2
Changed lines of the file:
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@@
+	(wire
+		(pts
+			(xy 29.21 41.91) (xy 43.18 41.91)
+		)
+		(stroke
+			(width 0)
+			(type default)
+		)
+	)
 	(wire
 		(pts
@@
 	(wire
 		(pts
-			(xy 63.5 52.07) (xy 63.5 60.96)
-		)
-		(stroke
-			(width 0)
-			(type default)
-		)
-	)
-	(wire
-		(pts
 			(xy 35.56 76.2) (xy 44.45 76.2)
 		)
@@
 	(wire
 		(pts
+			(xy 45.72 45.72) (xy 60.96 45.72)
+		)
+		(stroke
+			(width 0)
+			(type default)
+		)
+	)
+	(wire
+		(pts
 			(xy 139.7 62.23) (xy 139.7 72.39)
 		)
@@
 	(wire
 		(pts
+			(xy 43.18 52.07) (xy 45.72 52.07)
+		)
+		(stroke
+			(width 0)
+			(type default)
+		)
+	)
+	(wire
+		(pts
 			(xy 29.21 36.83) (xy 64.77 36.83)
 		)
@@
 	(wire
 		(pts
-			(xy 31.75 41.91) (xy 29.21 41.91)
-		)
-		(stroke
-			(width 0)
-			(type default)
-		)
-	)
-	(wire
-		(pts
 			(xy 123.19 46.99) (xy 153.67 46.99)
 		)
@@
 	(wire
 		(pts
-			(xy 45.72 52.07) (xy 38.1 52.07)
+			(xy 43.18 41.91) (xy 43.18 52.07)
 		)
 		(stroke
@@
 	(wire
 		(pts
-			(xy 31.75 60.96) (xy 31.75 41.91)
-		)
-		(stroke
-			(width 0)
-			(type default)
-		)
-	)
-	(wire
-		(pts
 			(xy 114.3 62.23) (xy 139.7 62.23)
 		)
@@
 	(wire
 		(pts
-			(xy 31.75 60.96) (xy 63.5 60.96)
+			(xy 45.72 39.37) (xy 45.72 45.72)
 		)
 		(stroke
@@
 	(wire
 		(pts
-			(xy 38.1 52.07) (xy 38.1 39.37)
-		)
-		(stroke
-			(width 0)
-			(type default)
-		)
-	)
-	(wire
-		(pts
 			(xy 38.1 95.25) (xy 30.48 95.25)
 		)
@@
 	(wire
 		(pts
+			(xy 60.96 45.72) (xy 60.96 52.07)
+		)
+		(stroke
+			(width 0)
+			(type default)
+		)
+	)
+	(wire
+		(pts
 			(xy 149.86 54.61) (xy 149.86 58.42)
 		)
@@
 	(wire
 		(pts
+			(xy 29.21 39.37) (xy 45.72 39.37)
+		)
+		(stroke
+			(width 0)
+			(type default)
+		)
+	)
+	(wire
+		(pts
 			(xy 114.3 59.69) (xy 144.78 59.69)
 		)
@@
 	(wire
 		(pts
-			(xy 63.5 52.07) (xy 60.96 52.07)
-		)
-		(stroke
-			(width 0)
-			(type default)
-		)
-	)
-	(wire
-		(pts
 			(xy 133.35 77.47) (xy 153.67 77.47)
 		)
@@
 		)
 		(stroke
-			(width 0)
-			(type default)
-		)
-	)
-	(wire
-		(pts
-			(xy 38.1 39.37) (xy 29.21 39.37)
-		)
-		(stroke
