File: Barboni!/Schema elettrificato/Norns/Norns.kicad_sch (KiCad schematic)
At the start: 38 parts, among them J1 Raspberry_Pi_4, J2 DIN-5, J3 DIN-5, J4 Power Supply, J5 Encoders, J6 Display, Q1 2N2222, Q3 2N2222, Q4 S8550, U1 NE555P, U2 7404, U3 6N138, U4 NE555P

Commit message: 2
Parts:
- removed J1: Raspberry_Pi_4, Connector_IDC:IDC-Header_2x20_P2.54mm_Vertical, symbol Connector:Raspberry_Pi_4
- removed J5: Encoders, Connector_JST:JST_EH_B12B-EH-A_1x12_P2.50mm_Vertical, symbol Connector:Conn_01x12_Pin
- added J7: RPi_GPIO, RPI_Hat:RPI_Hat_B+_NoCamera, symbol Raspberry Hat:RPi_GPIO
- added J8: Encoders, Connector_JST:JST_EH_B12B-EH-A_1x12_P2.50mm_Vertical, symbol Connector:Conn_01x12_Pin
- D2: value LED Blu -> LED Out; footprint Connector_PinHeader_2.54mm:PinHeader_1x02_P2.54mm_Vertical -> LED_THT:LED_D5.0mm
- D5: value LED Giallo -> LED In; footprint Connector_PinHeader_2.54mm:PinHeader_1x02_P2.54mm_Vertical -> LED_THT:LED_D5.0mm
- D7: value LED Verde (power on) -> LED Pwr; footprint Connector_PinHeader_2.54mm:PinHeader_1x02_P2.54mm_Vertical -> LED_THT:LED_D5.0mm
Connections:
- net +3.3V: now also J7.1 (3.3V), J8.1 (Pin_1)
- net +5V: now also J7.2 (5V)
- net CLK1: now also J7.7 (BCM4_GPCLK0), J8.9 (Pin_9)
- net CLK2: now also J7.18 (BCM24), J8.6 (Pin_6)
- net CLK3: now also J7.32 (BCM12_PWM0), J8.3 (Pin_3)
- net CS: now also J7.24 (BCM8_CE0)
- net Data1: now also J7.13 (BCM27), J8.10 (Pin_10)
- net Data2: now also J7.16 (BCM23), J8.7 (Pin_7)
- net Data3: now also J7.22 (BCM25), J8.4 (Pin_4)
- net GND: now also J7.14 (GND), J7.20 (GND), J7.25 (GND), J7.30 (GND), J7.34 (GND), J7.39 (GND), J7.6 (GND), J7.9 (GND), J8.12 (Pin_12)
- net MOSI: now also J7.19 (BCM10_MOSI)
- net O_DC: now also J7.29 (BCM5)
- net O_RESET: now also J7.31 (BCM6)
- net SCK: now also J7.23 (BCM11_SCLK)
- net SW1: now also J7.15 (BCM22), J8.11 (Pin_11)
- net SW2: now also J7.33 (BCM13_PWM1), J8.8 (Pin_8)
- net SW3: now also J7.37 (BCM26), J8.5 (Pin_5)
- net at U2.5: now also J7.40 (BCM21_SCLK_PCM_DO)
- net at R6.2, U2.8, U3.6 (VO2): now also J7.10 (BCM15_RXD)
- net at R14.1: now also J7.35 (BCM19_MISO_PCM_FS)
- net at U2.1: now also J7.8 (BCM14_TXD)
- no-connect marks 12 -> 23
Other:
- moved on the sheet: C1, C2, C3, C4, D1, D2, D3, D4, D5, D7, J2, J3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

Commit message: gerb
Parts:
- removed J2, J3: DIN-5, Connector_PinHeader_2.54mm:PinHeader_1x05_P2.54mm_Vertical, symbol Connector:DIN-5
- added J1, J2: MIDI_Din, Connector_PinHeader_2.54mm:PinHeader_1x02_P2.54mm_Vertical, symbol XOR Library:MIDI_Din
- C1, C4: footprint Capacitor_THT:C_Radial_D6.3mm_H11.0mm_P2.50mm -> Capacitor_THT:C_Radial_D5.0mm_H11.0mm_P2.00mm
- J7: footprint RPI_Hat:RPI_Hat_B+_NoCamera -> Raspoberro
- R11, R12, R13, R14, R15, R4, R5, R6, R7: footprint Resistor_THT:R_Axial_DIN0204_L3.6mm_D1.6mm_P7.62mm_Horizontal -> Resistor_THT:R_Axial_DIN0204_L3.6mm_D1.6mm_P5.08mm_Horizontal
Connections:
- net at D3.2 (A), U3.3 (C2): now also J2.2
- net at R12.2: now also J1.1
- net at R11.1: now also J1.2
- net at R5.2: now also J2.1
- net at J7.10 (BCM15_RXD), R6.2, U3.6 (VO2): now also U2.9; no longer U2.8
- net at R8.1: now also U2.8; no longer U2.9
- no-connect marks 23 -> 17
Other:
- note removed: "Visto da dietro"
- moved on the sheet: U2F

Commit message: avanzamento di progressione
Changed lines of the file:
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@@
 					(size 1.27 1.27)
 				)
-				(hide yes)
 			)
 		)
@@
 					(size 1.27 1.27)
 				)
-				(hide yes)
 			)
 		)

Commit message: schema el
Parts:
- removed C2, C3: 100nF, Capacitor_THT:C_Disc_D5.0mm_W2.5mm_P5.00mm, symbol Device:C_Small
- removed C4: 4,7mF, Capacitor_THT:C_Radial_D5.0mm_H11.0mm_P2.00mm, symbol Device:C_Polarized
- removed D1: 1N4148, Diode_THT:D_DO-35_SOD27_P7.62mm_Horizontal, symbol Diode:1N4148
- removed D2: LED Out, LED_THT:LED_D5.0mm, symbol Device:LED
- removed Q1: 2N2222, Package_TO_SOT_THT:TO-92_Inline, symbol XOR Library:2N2222
- removed Q3: 2N2222, Package_TO_SOT_THT:TO-92_Inline, symbol Transistor_BJT:MPSA42
- removed R1, R13, R3, R4: 1000, Resistor_THT:R_Axial_DIN0204_L3.6mm_D1.6mm_P5.08mm_Horizontal, symbol Device:R_US
- removed R2: 10000, Resistor_THT:R_Axial_DIN0204_L3.6mm_D1.6mm_P5.08mm_Horizontal, symbol Device:R_US
- removed U1, U4: NE555P, Package_DIP:DIP-8_W7.62mm, symbol Timer:NE555P
- added C2: 2,2 mF, Capacitor_THT:C_Radial_D5.0mm_H11.0mm_P2.00mm, symbol Device:C_Polarized
- added D3: 1N4148, Diode_THT:D_DO-35_SOD27_P7.62mm_Horizontal, symbol Diode:1N4148
- added D6: LED Out, LED_THT:LED_D5.0mm, symbol Device:LED
- added Q2, Q3: 2N7000, Package_TO_SOT_THT:TO-92_Inline, symbol Transistor_FET:2N7000
- added R11: 1000, Resistor_THT:R_Axial_DIN0204_L3.6mm_D1.6mm_P5.08mm_Horizontal, symbol Device:R_US
- C1: value 4,7mF -> 2,2 mF
- D5: value LED In -> LED Out
- J2: renamed from J7; footprint Raspoberro -> RPI_Hat:RPI_Hat_B+_NoCamera
- R10: value 10000 -> 1000
- R8, R9: value 1000 -> 100K
- renumbered D7 to D1, D3 to D2, J4 to J1, J6 to J3, J8 to J4, J2 to J5, J1 to J6, Q4 to Q1, R14 to R1, R7 to R2, R6 to R3, R15 to R4, R12 to R6, R11 to R7, U2 to U1, U3 to U2
Connections:
- net +5V: no longer R10.2, R9.2
- net GND: now also R8.1, R9.1, C2.2, D6.1 (K), Q2.1 (S), Q3.1 (S)
- net at C1.1: now also R8.2, D3.1 (K), Q2.2 (G)
- net at D4.1 (K): now also R9.2, C2.1, Q3.2 (G); no longer R9.1
- net at R10.1: now also Q2.3 (D); no longer D4.2 (A)
- net at U1.2, U1.3: now also D3.2 (A)
- net at U1.8: now also D4.2 (A); no longer R8.1
- net at D5.2 (A): now also R10.2
- new net: Q3.3 (D), R11.1
- new net: D6.2 (A), R11.2

Commit message: a
Parts:
- removed J3: Display, Connector_JST:JST_EH_B8B-EH-A_1x08_P2.50mm_Vertical, symbol Connector_Generic:Conn_01x08
- removed J4: Encoders, Connector_JST:JST_EH_B12B-EH-A_1x12_P2.50mm_Vertical, symbol Connector:Conn_01x12_Pin
- added J1: Display, Connector_JST:JST_EH_B8B-EH-A_1x08_P2.50mm_Vertical, symbol Connector_Generic:Conn_01x08
- added J2: Encoder 1, Connector_JST:JST_EH_B5B-EH-A_1x05_P2.50mm_Vertical, symbol Connector_Generic:Conn_01x05
- added J5: Encoder 2, Connector_JST:JST_EH_B5B-EH-A_1x05_P2.50mm_Vertical, symbol Connector_Generic:Conn_01x05
- added J6: Encoder 3, Connector_JST:JST_EH_B5B-EH-A_1x05_P2.50mm_Vertical, symbol Connector_Generic:Conn_01x05
- renumbered C2 to C1, C1 to C2, D4 to D3, D3 to D4, D6 to D5, D5 to D6, J1 to J3, J2 to J4, J5 to J7, J6 to J8, Q3 to Q2, Q2 to Q3, R11 to R10, R10 to R11, R9 to R8, R8 to R9
Connections:
- net +3.3V: now also J1.1 (Pin_1), J2.1 (Pin_1), J5.1 (Pin_1), J6.1 (Pin_1)
- net +5V: now also R10.2, R11.2
- net CS: now also J1.2 (Pin_2)
- net Data2: now also J5.2 (Pin_2)
- net Data3: now also J6.2 (Pin_2)
- net GND: now also J1.8 (Pin_8), J2.5 (Pin_5), J5.5 (Pin_5), J6.5 (Pin_5); no longer D5.1 (K), D6.1 (K)
- net LED_BL: now also J1.7 (Pin_7)
- net MOSI: now also J1.4 (Pin_4)
- net O_DC: now also J1.6 (Pin_6)
- net O_RESET: now also J1.3 (Pin_3)
- net SCK: now also J1.5 (Pin_5)
- net at Q2.3 (D): now also D5.1 (K); no longer R10.1
- net at D5.2 (A): now also R10.1; no longer R10.2
- net at D6.2 (A): now also R11.1; no longer R11.2
- net at Q3.3 (D): now also D6.1 (K); no longer R11.1
- net CLK1 renamed Clock
- net Clock: now also J2.3 (Pin_3)
- net CLK2 renamed Clk2
- net Clk2: now also J5.3 (Pin_3)
- net CLK3 renamed Clk3
- net Clk3: now also J6.3 (Pin_3)
- net Data1 renamed Data
- net Data: now also J2.2 (Pin_2)
- net SW1 renamed Switch
- net Switch: now also J2.4 (Pin_4)
- net SW2 renamed Switch2
- net Switch2: now also J5.4 (Pin_4)
- net SW3 renamed Switch3
- net Switch3: now also J6.4 (Pin_4)
- no-connect marks 17 -> 16
Other:
- moved on the sheet: C1, C2, D1, D2, D3, D4, D5, D6, J3, J4, J7, J8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

Commit message: modifiche
Parts:
- removed D1: LED Pwr, LED_THT:LED_D5.0mm, symbol Device:LED
- removed D5, D6: LED Out, LED_THT:LED_D5.0mm, symbol Device:LED
- removed J2: Encoder 1, Connector_JST:JST_EH_B5B-EH-A_1x05_P2.50mm_Vertical, symbol Connector_Generic:Conn_01x05
- removed J5: Encoder 2, Connector_JST:JST_EH_B5B-EH-A_1x05_P2.50mm_Vertical, symbol Connector_Generic:Conn_01x05
- removed J6: Encoder 3, Connector_JST:JST_EH_B5B-EH-A_1x05_P2.50mm_Vertical, symbol Connector_Generic:Conn_01x05
- removed J7, J8: MIDI_Din, Connector_PinHeader_2.54mm:PinHeader_1x02_P2.54mm_Vertical, symbol XOR Library:MIDI_Din
- added J4: Encoders, Connector_JST:JST_EH_B12B-EH-A_1x12_P2.50mm_Vertical, symbol Connector_Generic:Conn_01x12
- added J5: MIDI, Connector_JST:JST_EH_B4B-EH-A_1x04_P2.50mm_Vertical, symbol Connector_Generic:Conn_01x04
- added J6: LED, Connector_JST:JST_EH_B6B-EH-A_1x06_P2.50mm_Vertical, symbol Connector_Generic:Conn_01x06
- J2: renamed from J4; value RPi_GPIO -> Raspoberro; footprint RPI_Hat:RPI_Hat_B+_NoCamera -> RPI_Hat:RPI_Hat_B+_No_Camera
- renumbered D2 to D1, D3 to D2, D4 to D3
Connections:
- net +3.3V: now also J4.1 (Pin_1)
- net GND: now also J4.12 (Pin_12), J6.6 (Pin_6)
- net at D1.2 (A), U2.3 (C2): now also J5.4 (Pin_4)
- net at R6.2: now also J5.1 (Pin_1)
- net at R7.1: now also J5.2 (Pin_2)
- net at Q2.3 (D): now also J6.4 (Pin_4)
- net at R2.1: now also J6.5 (Pin_5)
- net at R5.2: now also J5.3 (Pin_3)
- net at R10.1: now also J6.3 (Pin_3)
- net at Q3.3 (D): now also J6.2 (Pin_2)
- net at R11.1: now also J6.1 (Pin_1)
- net Clk2: no longer names the net of J2.18 (BCM24)
- net Clk2: now also J4.6 (Pin_6)
- net Clk3: no longer names the net of J2.32 (BCM12_PWM0)
- net Clk3: now also J4.9 (Pin_9)
- net Clock: no longer names the net of J2.7 (BCM4_GPCLK0)
- net Clock: now also J4.3 (Pin_3)
- net Data: no longer names the net of J2.13 (BCM27)
- net Data: now also J4.2 (Pin_2)
- net Data2: no longer names the net of J2.16 (BCM23)
- net Data2: now also J4.5 (Pin_5)
- net Data3: no longer names the net of J2.22 (BCM25)
- net Data3: now also J4.8 (Pin_8)
- net Switch: no longer names the net of J2.15 (BCM22)
- net Switch: now also J4.4 (Pin_4)
- net Switch2: no longer names the net of J2.33 (BCM13_PWM1)
- net Switch2: now also J4.7 (Pin_7)
- net Switch3: no longer names the net of J2.37 (BCM26)
- net Switch3: now also J4.10 (Pin_10)
- no-connect marks 16 -> 17
Other:
- note removed: "MIDI IN"
- note removed: "MIDI OUT"
- moved on the sheet: J3, R10, R11, R7, U1E, U1F

Commit message: ola
Other:
- moved on the sheet: D2
Changed lines of the file:
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@@
 	)
 	(junction
-		(at 227.33 143.51)
-		(diameter 0)
-		(color 0 0 0 0)
-	)
-	(junction
 		(at 240.03 143.51)
 		(diameter 0)
@@
 	(wire
 		(pts
-			(xy 240.03 143.51) (xy 233.68 143.51)
+			(xy 234.95 143.51) (xy 240.03 143.51)
 		)
 		(stroke
@@
 	(wire
 		(pts
-			(xy 227.33 143.51) (xy 228.6 143.51)
-		)
-		(stroke
-			(width 0)
-			(type default)
-		)
-	)
-	(wire
-		(pts
 			(xy 116.84 105.41) (xy 113.03 105.41)
 		)
@@
 	(wire
 		(pts
-			(xy 227.33 143.51) (xy 226.06 143.51)
-		)
-		(stroke
-			(width 0)
-			(type default)
-		)
-	)
-	(wire
-		(pts
 			(xy 50.8 34.29) (xy 137.16 34.29)
 		)
@@
 	(symbol
 		(lib_id "Diode:1N4148")
-		(at 229.87 143.51 180)
+		(at 231.14 143.51 180)
 		(unit 1)
 		(body_style 1)
@@
 		(dnp no)
 		(property "Reference" "D2"
-			(at 229.87 149.86 0)
+			(at 231.14 149.86 0)
 			(show_name no)
 			(do_not_autoplace no)
@@
 		)
 		(property "Value" "1N4148"
-			(at 230.378 146.812 0)
+			(at 231.648 146.812 0)
 			(show_name no)
 			(do_not_autoplace no)
@@
 		)
 		(property "Footprint" "Diode_THT:D_DO-35_SOD27_P7.62mm_Horizontal"
-			(at 229.87 143.51 0)
+			(at 231.14 143.51 0)
 			(hide yes)
 			(show_name no)
@@
 		)
 		(property "Datasheet" "https://assets.nexperia.com/documents/data-sheet/1N4148_1N4448.pdf"
-			(at 229.87 143.51 0)
+			(at 231.14 143.51 0)
 			(hide yes)
 			(show_name no)
@@
 		)
 		(property "Description" "100V 0.15A standard switching diode, DO-35"
-			(at 229.87 143.51 0)
+			(at 231.14 143.51 0)
 			(hide yes)
 			(show_name no)
@@
 		)
 		(property "Sim.Device" "D"
-			(at 229.87 143.51 0)
+			(at 231.14 143.51 0)
 			(hide yes)
 			(show_name no)
@@
 		)
 		(property "Sim.Pins" "1=K 2=A"
-			(at 229.87 143.51 0)
+			(at 231.14 143.51 0)
 			(hide yes)
 			(show_name no)
@@
 		)
 		(property "Sim.Type" ""
-			(at 229.87 143.51 0)
+			(at 231.14 143.51 0)
 			(hide yes)
 			(show_name no)

Commit message: committamento
Parts:
- C1, C2: footprint Capacitor_THT:C_Radial_D5.0mm_H11.0mm_P2.00mm -> Capacitor_THT:CP_Radial_D5.0mm_P2.50mm
- U2: footprint Package_DIP:DIP-8_W7.62mm_LongPads -> Package_DIP:DIP-8_W7.62mm
Changed lines of the file:
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@@
 			)
 		)
-		(property "Footprint" "Capacitor_THT:C_Radial_D5.0mm_H11.0mm_P2.00mm"
+		(property "Footprint" "Capacitor_THT:CP_Radial_D5.0mm_P2.50mm"
 			(at 242.2652 82.55 0)
 			(hide yes)
@@
 			)
 		)
-		(property "Footprint" "Capacitor_THT:C_Radial_D5.0mm_H11.0mm_P2.00mm"
+		(property "Footprint" "Capacitor_THT:CP_Radial_D5.0mm_P2.50mm"
 			(at 240.9952 151.13 0)
 			(hide yes)
@@
 			)
 		)
-		(property "Footprint" "Package_DIP:DIP-8_W7.62mm_LongPads"
+		(property "Footprint" "Package_DIP:DIP-8_W7.62mm"
 			(at 190.754 118.11 0)
 			(hide yes)
