File: Barboni!/Schema elettrificato/Norns/Norns.kicad_sch (KiCad schematic)
At the start: 27 parts, among them J1 Display, J2 Raspoberro, J3 Power Supply, J4 Encoders, J5 MIDI, J6 LED, Q1 S8550, Q2 2N7000, Q3 2N7000, U1 7404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

Commit message: pcb
Other:
- title: (none) -> Trapanaorecchie
Changed lines of the file:
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@@
 	(generator_version "10.0")
 	(paper "A4")
+	(title_block
+		(title "Trapanaorecchie")
+		(date "2026-06-05")
+		(rev "1.0")
+		(comment 1 "Una libera reinterpretazione del Monome Norns")
+	)
 	(junction
 		(at 241.3 74.93)
